File: HapticGPS/HapticGPS.kicad_pcb (KiCad board)
At the start: 2 copper layers, 1 part

Commit message: updating
Parts:
- added AE1: Antenna, RF_Antenna:Texas_SWRA117D_2.4GHz_Left, F.Cu at (144.4, 68.3)
- added C1: 10uF, Capacitor_SMD:C_0603_1608Metric, F.Cu at (101.7, 72.5)
- added C10: 100nF, Capacitor_SMD:C_0603_1608Metric, F.Cu at (129.6, 68.4)
- added C11: 100nF, Capacitor_SMD:C_0603_1608Metric, F.Cu at (129.6, 70.9)
- added C12: 100nF, Capacitor_SMD:C_0603_1608Metric, F.Cu at (129.6, 73.4)
- added C13: 7pF, Capacitor_SMD:C_0402_1005Metric, F.Cu at (133.0, 70.2)
- added C14: 7pF, Capacitor_SMD:C_0402_1005Metric, F.Cu at (133.0, 72.2)
- added C15: 1.5pF, Capacitor_SMD:C_0201_0603Metric, F.Cu at (135.7, 70.1)
- added C16: 2pF, Capacitor_SMD:C_0201_0603Metric, F.Cu at (135.7, 71.8)
- added C17: 100nF, Capacitor_SMD:C_0603_1608Metric, F.Cu at (101.7, 85.0)
- added C18: 100nF, Capacitor_SMD:C_0603_1608Metric, F.Cu at (101.7, 92.0)
- added C19: 100nF, Capacitor_SMD:C_0603_1608Metric, F.Cu at (101.7, 94.5)
- added C2: 10uF, Capacitor_SMD:C_0603_1608Metric, F.Cu at (101.7, 75.0)
- added C20: 10nF, Capacitor_SMD:C_0603_1608Metric, F.Cu at (101.7, 97.1)
- added C21: 10nF, Capacitor_SMD:C_0603_1608Metric, F.Cu at (101.7, 99.6)
- added C22: 4.7uF, Capacitor_SMD:C_0603_1608Metric, F.Cu at (152.2, 85.9)
- added C23: 4.7uF, Capacitor_SMD:C_0603_1608Metric, F.Cu at (152.2, 88.4)
- added C24: 1uF, Capacitor_SMD:C_0603_1608Metric, F.Cu at (152.2, 63.4)
- added C25: 10uF, Capacitor_SMD:C_0805_2012Metric, F.Cu at (161.4, 76.0)
- added C26: 100nF, Capacitor_SMD:C_0603_1608Metric, F.Cu at (152.2, 65.9)
- added C27: 100nF, Capacitor_SMD:C_0603_1608Metric, F.Cu at (152.2, 68.4)
- added C28: 100nF, Capacitor_SMD:C_0603_1608Metric, F.Cu at (152.2, 70.9)
- added C29: 2pF, Capacitor_SMD:C_0201_0603Metric, F.Cu at (135.7, 73.6)
- added C3: 2.2uF, Capacitor_SMD:C_0603_1608Metric, F.Cu at (101.7, 77.5)
- added C30: 10uF, Capacitor_SMD:C_0805_2012Metric, F.Cu at (139.1, 77.7)
- added C31: 2.2uF, Capacitor_SMD:C_0402_1005Metric, F.Cu at (133.0, 74.1)
- added C32: 10nF, Capacitor_SMD:C_0402_1005Metric, F.Cu at (133.0, 76.1)
- added C33: 2.2nF, Capacitor_SMD:C_0402_1005Metric, F.Cu at (133.0, 78.1)
- added C34: 2.2uF, Capacitor_SMD:C_0402_1005Metric, F.Cu at (133.0, 80.0)
- added C35: 20pF, Capacitor_SMD:C_0402_1005Metric, F.Cu at (133.0, 82.0)
- added C36: 20pF, Capacitor_SMD:C_0402_1005Metric, F.Cu at (133.0, 84.0)
- added C37: 100nF, Capacitor_SMD:C_0603_1608Metric, F.Cu at (129.6, 75.9)
- added C4: 100nF, Capacitor_SMD:C_0603_1608Metric, F.Cu at (101.7, 89.5)
- added C5: 10uF, Capacitor_SMD:C_0805_2012Metric, F.Cu at (114.9, 80.0)
- added C6: 100nF, Capacitor_SMD:C_0603_1608Metric, F.Cu at (101.7, 80.0)
- added C7: 1uF, Capacitor_SMD:C_0603_1608Metric, F.Cu at (101.7, 82.5)
- added C8: 100nF, Capacitor_SMD:C_0603_1608Metric, F.Cu at (129.6, 63.4)
- added C9: 100nF, Capacitor_SMD:C_0603_1608Metric, F.Cu at (129.6, 65.9)
- added D1: GREEN, LED_SMD:LED_0402_1005Metric, F.Cu at (114.3, 82.5)
- added FB1: BLM18AG, Inductor_SMD:L_0603_1608Metric, F.Cu at (129.6, 78.4)
- added IC1: BOS1921CQR, Package_DFN_QFN:VQFN-24-1EP_4x4mm_P0.5mm_EP2.45x2.45mm_ThermalVias, F.Cu at (107.2, 98.0)
- added J2: PZ, Connector_PinSocket_2.00mm:PinSocket_1x02_P2.00mm_Vertical, F.Cu at (112.4, 96.8)
- added J3: Conn_01x02, Connector_PinSocket_2.00mm:PinSocket_1x02_P2.00mm_Vertical, F.Cu at (156.3, 64.1)
- added J4: Conn_01x02, Connector_PinSocket_2.00mm:PinSocket_1x02_P2.00mm_Vertical, F.Cu at (160.3, 64.1)
- added L1: 2.2uF, Inductor_SMD:L_1008_2520Metric, F.Cu at (110.2, 80.4)
- added L2: 2.2uF, Inductor_SMD:L_1008_2520Metric, F.Cu at (110.2, 84.2)
- added L3: 2.7nH, Inductor_SMD:L_0201_0603Metric, F.Cu at (135.7, 75.3)
- added L4: 3.5nH, Inductor_SMD:L_0201_0603Metric, F.Cu at (135.7, 77.1)
- added L5: 3.5nH, Inductor_SMD:L_0201_0603Metric, F.Cu at (135.7, 78.8)
- added L6: 22uH, Inductor_SMD:L_Taiyo-Yuden_MD-5050, F.Cu at (107.0, 91.5)
- added L7: 2.2uF, Inductor_SMD:L_1008_2520Metric, F.Cu at (156.7, 76.3)
- added L8: 4.7uH, Inductor_SMD:L_0603_1608Metric, F.Cu at (129.6, 80.9)
- added R1: 2.2k, Capacitor_SMD:C_0603_1608Metric, F.Cu at (105.7, 72.5)
- added R10: 7.68K, Resistor_SMD:R_0603_1608Metric, F.Cu at (152.2, 78.4)
- added R2: 2.2k, Capacitor_SMD:C_0603_1608Metric, F.Cu at (105.7, 75.0)
- added R3: 2.2k, Capacitor_SMD:C_0603_1608Metric, F.Cu at (105.7, 77.5)
- added R4: 100K, Resistor_SMD:R_0603_1608Metric, F.Cu at (105.7, 80.0)
- added R5: 100K, Resistor_SMD:R_0603_1608Metric, F.Cu at (105.7, 82.5)
- added R6: 0.5, Resistor_SMD:R_0805_2012Metric, F.Cu at (112.5, 89.8)
- added R7: 1, Resistor_SMD:R_0805_2012Metric, F.Cu at (152.4, 83.2)
- added R8: 510k, Resistor_SMD:R_0603_1608Metric, F.Cu at (152.2, 73.4)
- added R9: 37k, Resistor_SMD:R_0603_1608Metric, F.Cu at (152.2, 75.9)
- added U1: NPM1300, Package_DFN_QFN:VQFN-32-1EP_5x5mm_P0.5mm_EP3.1x3.1mm_ThermalVias, F.Cu at (111.7, 74.9)
- added U2: NRF54L15-QFAA-R, Package_DFN_QFN:QFN-48-1EP_6x6mm_P0.4mm_EP4.6x4.6mm_ThermalVias, F.Cu at (121.2, 92.4)
- added U3: DRV2667RGPR, Package_DFN_QFN:Texas_RGP0020D_VQFN-20-1EP_4x4mm_P0.5mm_EP2.7x2.7mm_ThermalVias, F.Cu at (157.8, 71.3)
- added U4: CY15B108, Package_SO:SOIC-8_5.3x5.3mm_P1.27mm, F.Cu at (142.1, 72.7)
- added Y1: 32MHz, Crystal:Crystal_SMD_2016-4Pin_2.0x1.6mm, F.Cu at (118.8, 98.3)
- added Y2: 32kHz, Crystal:Crystal_SMD_2012-2Pin_2.0x1.2mm, F.Cu at (138.9, 80.8)

Commit message: save
Parts:
- removed the C10 at (129.6, 68.4)
- removed the C11 at (129.6, 70.9)
- removed the C12 at (129.6, 73.4)
- removed the U1 at (146.4, 107.8)
- removed the U1 at (111.7, 74.9)
- added AE2: ANT-GNCP, Sadman_antenna:NT-GNCP-TH258L15, F.Cu at (263.8, 71.0)
- added C10: 100nF, Capacitor_SMD:C_0402_1005Metric, F.Cu at (174.1, 137.2)
- added C10: 100nF, Capacitor_SMD:C_0603_1608Metric, F.Cu at (145.6, 61.9)
- added C11: 100nF, Capacitor_SMD:C_0603_1608Metric, F.Cu at (145.6, 64.4)
- added C11: 100nF, Capacitor_SMD:C_0402_1005Metric, F.Cu at (168.1, 135.0)
- added C12: 100nF, Capacitor_SMD:C_0402_1005Metric, F.Cu at (169.7, 128.8)
- added C12: 100nF, Capacitor_SMD:C_0603_1608Metric, F.Cu at (145.6, 66.9)
- added C38: 10uF, Capacitor_SMD:C_0805_2012Metric, B.Cu at (278.7, 49.2)
- added C39: 100nF, Capacitor_SMD:C_0603_1608Metric, B.Cu at (276.9, 49.4)
- added C40: 33pF, Capacitor_SMD:C_0402_1005Metric, B.Cu at (275.5, 49.9)
- added C41: 4.7uF, Capacitor_SMD:C_0603_1608Metric, B.Cu at (271.5, 49.4)
- added C42: 100nF, Capacitor_SMD:C_0603_1608Metric, B.Cu at (273.0, 49.4)
- added C43: 33pF, Capacitor_SMD:C_0402_1005Metric, B.Cu at (274.4, 49.9)
- added C44: 220mF, sadman_power_passive:FC0H224ZFTBR24, B.Cu at (254.5, 60.5)
- added C45: 2pF, Capacitor_SMD:C_0402_1005Metric, B.Cu at (264.2, 68.2)
- added C46: 2pF, Capacitor_SMD:C_0402_1005Metric, B.Cu at (263.3, 70.8)
- added C47: 100nF, Capacitor_SMD:C_0603_1608Metric, B.Cu at (260.7, 46.2)
- added C48: 100nF, Capacitor_SMD:C_0603_1608Metric, B.Cu at (258.2, 43.2)
- added D2: TVS, Diode_SMD:D_0402_1005Metric, B.Cu at (279.6, 52.0)
- added D3: TVS, Diode_SMD:D_0402_1005Metric, B.Cu at (269.3, 50.1)
- added D4: 1N4148WT, Diode_SMD:D_SOD-523, B.Cu at (249.9, 51.5)
- added D5: TVS, Diode_SMD:D_0201_0603Metric, B.Cu at (264.1, 71.6)
- added D6: YELLOW, Diode_SMD:D_0402_1005Metric, B.Cu at (249.6, 49.0)
- added J5: Conn_01x10, Connector_FFC-FPC:Amphenol_F32Q-1A7x1-11010_1x10-1MP_P0.5mm_Horizontal, F.Cu at (265.0, 40.5)
- added L9: 6nH, Inductor_SMD:L_0402_1005Metric, B.Cu at (263.8, 69.5)
- added Q1: RU1J002, Package_TO_SOT_SMD:SOT-323_SC-70, B.Cu at (253.9, 46.1)
- added R11: 2.2k, Capacitor_SMD:C_0603_1608Metric, F.Cu at (150.3, 153.6)
- added R12: 1k, Resistor_SMD:R_0603_1608Metric, B.Cu at (252.8, 51.5)
- added R13: 1, Resistor_SMD:R_0805_2012Metric, B.Cu at (251.8, 40.5)
- added R14: 2.2k, Capacitor_SMD:C_0603_1608Metric, B.Cu at (279.1, 65.7)
- added R15: 100K, Resistor_SMD:R_0603_1608Metric, B.Cu at (279.1, 62.2)
- added R16: 75, Resistor_SMD:R_0603_1608Metric, B.Cu at (251.3, 48.5)
- added R17: 2.2k, Capacitor_SMD:C_0603_1608Metric, B.Cu at (276.7, 68.9)
- added R18: 2.2k, Capacitor_SMD:C_0603_1608Metric, B.Cu at (267.1, 68.9)
- added R19: 1, Resistor_SMD:R_0805_2012Metric, B.Cu at (251.8, 42.8)
- added R20: 2.2k, Capacitor_SMD:C_0603_1608Metric, B.Cu at (256.6, 43.2)
- added R21: 2.2k, Capacitor_SMD:C_0603_1608Metric, B.Cu at (263.8, 44.9)
- added R22: 1k, Resistor_SMD:R_0603_1608Metric, F.Cu at (156.0, 66.5)
- added U1: NPM1300, Package_DFN_QFN:VQFN-32-1EP_5x5mm_P0.5mm_EP3.1x3.1mm_ThermalVias, B.Cu at (161.4, 106.6)
- added U5: LC29H, Sadman_RF_receivers:LC29H, B.Cu at (262.6, 59.2)
- added U6: LSM6, Package_LGA:LGA-14_3x2.5mm_P0.5mm_LayoutBorder3x4y, B.Cu at (261.2, 43.2)
- added U7: TPS22917DBV, Package_TO_SOT_SMD:SOT-23-6, F.Cu at (156.6, 63.0)
- C1, C17, C2, C5, C6, L1, L2, R4, R5: moved to B.Cu
- C3: footprint Capacitor_SMD:C_0603_1608Metric -> Capacitor_SMD:C_0402_1005Metric; moved to B.Cu
- C8, C9: footprint Capacitor_SMD:C_0603_1608Metric -> Capacitor_SMD:C_0402_1005Metric
- moved C7 98.8 mm to (149.0, 169.3)
- moved R2 98.8 mm to (153.0, 161.7)
- moved R3 98.8 mm to (153.0, 164.2)
- moved R1 98.8 mm to (153.0, 159.2)
- moved D1 97.1 mm to (171.7, 160.9)
- moved C9 77.6 mm to (175.2, 128.6), turned to 90 degrees
- moved C8 76.8 mm to (168.4, 129.6), turned to 90 degrees
- moved C16 75.1 mm to (178.9, 133.3), turned to -90 degrees
- moved U4 74.6 mm to (172.2, 141.0)
- moved C15 74.5 mm to (176.5, 132.4), turned to 180 degrees
- moved C29 74.2 mm to (180.6, 132.7), turned to 90 degrees
- moved C13 74.0 mm to (178.9, 128.2), turned to 90 degrees
- moved L3 70.7 mm to (176.6, 133.0)
- moved C3 70.7 mm to (165.9, 106.9)
- moved C32 70.3 mm to (176.9, 130.9), turned to 90 degrees
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Connections:
- C1 pad 1: +3VDC2 -> +3VDC1
- C17 pad 1: +3VDC2 -> +3VDC1
- C30 pad 1: Net-(U2-VDD) -> +3VDC1
- C8 pad 1: Net-(U2-VDD) -> +3VDC1
- C9 pad 1: Net-(U2-VDD) -> +3VDC1
- L1 pad 1: Net-(U1-SW1) -> /POWER/SW1_NPM
- L1 pad 2: +3VDC2 -> +3VDC1
- U2 pad 10: Net-(U2-VDD) -> +3VDC1
- U2 pad 22: Net-(U2-VDD) -> +3VDC1
- U2 pad 36: Net-(U2-VDD) -> +3VDC1
- U2 pad 47: Net-(U2-VDD) -> +3VDC1
- U2 pad 48: Net-(U2-VDD) -> +3VDC1
Routing:
- net GND: track 0.00 -> 64.6 mm, vias 0 -> 68
- net /GPS_NRST: track 0.00 -> 60.4 mm, vias 0 -> 1
- net /GPS_WK: track 0.00 -> 49.9 mm, vias 0 -> 1
- net Net-(Q1-G): track 0.00 -> 39.8 mm, vias 0 -> 2
- net +3VDC1: track 0.00 -> 21.0 mm, vias 0 -> 6
- net /GPS_TX: track 0.00 -> 18.4 mm, vias 0 -> 1
- net /GPS_RX: track 0.00 -> 17.0 mm, vias 0 -> 1
- net /IMU_INT2: track 0.00 -> 12.3 mm, vias 0 -> 1
- net Net-(U6-CS): track 0.00 -> 11.4 mm
- net +3VDC2: track 0.00 -> 10.4 mm, vias 0 -> 2
- net Net-(U5-1PPS): track 0.00 -> 7.73 mm
- net /SCL_OUT: track 0.00 -> 7.44 mm, vias 0 -> 1
- net /SDA_OUT: track 0.00 -> 7.28 mm, vias 0 -> 1
- net /CONTROLLER/NRF_DECA: track 0.00 -> 7.23 mm, vias 0 -> 2
- net /CONTROLLER/NRF_XC2: track 0.00 -> 6.31 mm
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- added copper zone on B.Cu, net /GPS_INTERFACE/VBACKUP_GPS
- added copper zone on B.Cu, net /VINC_GPS
- added copper zone on F.Cu, net /VINC_GPS
- added copper zone on In2.Cu, net /VINC_GPS
- added copper zone on B.Cu, net GND
- added copper zone on F.Cu, net GND
- added copper zone on In1.Cu, net GND
- added copper zone on In2.Cu, net GND
Other:
- board outline added: 35 x 50 mm
- copper layers 2 -> 4
