File: HapticGPS/modules/controller.sch.kicad_sch (KiCad schematic)
At the start: 29 parts, among them U2 NRF54L15-QFAA-R, U4 CY15B108, Y1 32MHz, Y2 32kHz

Commit message: save
Parts:
- C10, C11, C12, C8, C9: footprint Capacitor_SMD:C_0603_1608Metric -> Capacitor_SMD:C_0402_1005Metric; Manufacturer KEMET -> Murata Electronics; Number Part C0603C104K3RACTU -> GCM155R71H104KE02J

Commit message: eliminating GPS, and second piezo driver
Parts:
- added D2: GREEN, LED_SMD:LED_0402_1005Metric, symbol Device:LED
- added J1: Conn_01x01, Connector_PinHeader_2.00mm:PinHeader_1x01_P2.00mm_Vertical, symbol Connector_Generic:Conn_01x01
- added J3: Conn_02x02_Counter_Clockwise, symbol Connector_Generic:Conn_02x02_Counter_Clockwise
- added R8: 120, Resistor_SMD:R_0402_1005Metric, symbol Device:R
- AE1: now left out of the parts list
- C15: footprint Capacitor_SMD:C_0201_0603Metric -> Capacitor_SMD:C_0402_1005Metric; Number Part GJM0335C1E1R5WB01J -> GRM1555C1H1R5CA01D
- C16, C29: footprint Capacitor_SMD:C_0201_0603Metric -> Capacitor_SMD:C_0402_1005Metric; Number Part GJM0335C1E2R0WB01D -> GJM1555C1H2R0WB01D
- L3: footprint Inductor_SMD:L_0201_0603Metric -> Inductor_SMD:L_0402_1005Metric; Number Part LQP03HQ2N7B02D -> LQG15HS2N7S02D
- L4, L5: footprint Inductor_SMD:L_0201_0603Metric -> Inductor_SMD:L_0402_1005Metric; Number Part LQP03HQ3N5B02D -> LQG15WH3N5B02D
- R11: footprint Capacitor_SMD:C_0603_1608Metric -> Resistor_SMD:R_0603_1608Metric
- U2: Manufacturer (none) -> Nordic Semiconductor ASA; Number Part (none) -> NRF54L15-QFAA-R; Provider (none) -> Digikey; Revisado (none) -> REV; STANDARD IPC-7351B -> (none); sad (none) -> IPC-7351B
- Y2: value 32kHz -> 32.768kHz
Connections:
- net GND: now also D2.1 (K), J1.1 (Pin_1)
- net NRF_CSMEMORY: now also U2.17 (P2.06/TRACECLK)
- net NRF_MISO: now also U2.16 (P2.05)
- net NRF_MOSI: now also U2.14 (P2.03)
- net NRF_RESET: now also J3.2 (Pin_2)
- net NRF_SCK: now also U2.15 (P2.04)
- net NRF_SWDCLK: now also J3.4 (Pin_4)
- net NRF_SWDIO: now also J3.3 (Pin_3)
- net NRF_VIN: now also C37.1, U4.8 (VDD)
- net NRF_WPMEMORY: now also U2.13 (P2.02)
- net at U2.19 (P2.08/TRACEDATA(1)): now also R8.2
- net SCL: now reaches U2.37 (P1.09/ASO(2)/RADIO(0))
- net SDA: now reaches U2.38 (P1.10/ASI(2)/RADIO(1))
- net NRF_INT: now reaches U2.7 (P1.06/ASO(1)/AIN2)
- new net: D2.2 (A), R8.1
- new net VIN: J3.1 (Pin_1)
